Commit message: test: add full vcan diffbot launch coverage

File: src/vcan_diffbot_demo/urdf/diffbot.urdf.xacro (robot description, xacro)
@@ -12,4 +12,9 @@
     <color rgba="0.08 0.08 0.08 1.0"/>
   </material>
+  <link name="base_footprint"/>
+  <joint name="base_footprint_joint" type="fixed">
+    <parent link="base_footprint"/>
+    <child link="base_link"/>
+  </joint>
   <link name="base_link">
     <visual>
