Commit message: feat: share motor configuration across CAN endpoints

File: src/vcan_diffbot_demo/urdf/diffbot.ros2_control.xacro (robot description, xacro)
@@ -1,14 +1,14 @@
 <?xml version="1.0"?>
 <robot xmlns:xacro="http://www.ros.org/wiki/xacro">
-  <xacro:macro name="vcan_diffbot_ros2_control" params="name can_interface">
+  <xacro:macro name="vcan_diffbot_ros2_control" params="name can_interface left_node_id right_node_id encoder_counts_per_revolution command_watchdog_ms feedback_timeout_ms">
     <ros2_control name="${name}" type="system">
       <hardware>
         <plugin>vcan_diffbot_demo/CanMotorHardware</plugin>
         <param name="can_interface">${can_interface}</param>
-        <param name="left_node_id">1</param>
-        <param name="right_node_id">2</param>
-        <param name="encoder_counts_per_revolution">4096</param>
-        <param name="command_watchdog_ms">200</param>
-        <param name="feedback_timeout_ms">500</param>
+        <param name="left_node_id">${left_node_id}</param>
+        <param name="right_node_id">${right_node_id}</param>
+        <param name="encoder_counts_per_revolution">${encoder_counts_per_revolution}</param>
+        <param name="command_watchdog_ms">${command_watchdog_ms}</param>
+        <param name="feedback_timeout_ms">${feedback_timeout_ms}</param>
       </hardware>
       <joint name="left_wheel_joint">

File: src/vcan_diffbot_demo/urdf/diffbot.urdf.xacro (robot description, xacro)
@@ -2,4 +2,9 @@
 <robot xmlns:xacro="http://www.ros.org/wiki/xacro" name="vcan_diffbot">
   <xacro:arg name="can_interface" default="vcan0"/>
+  <xacro:arg name="left_node_id" default="1"/>
+  <xacro:arg name="right_node_id" default="2"/>
+  <xacro:arg name="encoder_counts_per_revolution" default="4096"/>
+  <xacro:arg name="command_watchdog_ms" default="200"/>
+  <xacro:arg name="feedback_timeout_ms" default="500"/>
   <xacro:property name="wheel_radius" value="0.10"/>
   <xacro:property name="wheel_width" value="0.05"/>
@@ -76,4 +81,9 @@
   <xacro:vcan_diffbot_ros2_control
     name="VcanDiffBot"
-    can_interface="$(arg can_interface)"/>
+    can_interface="$(arg can_interface)"
+    left_node_id="$(arg left_node_id)"
+    right_node_id="$(arg right_node_id)"
+    encoder_counts_per_revolution="$(arg encoder_counts_per_revolution)"
+    command_watchdog_ms="$(arg command_watchdog_ms)"
+    feedback_timeout_ms="$(arg feedback_timeout_ms)"/>
 </robot>

Commit message: fix: separate ACK deadline and clarify workflow

File: src/vcan_diffbot_demo/urdf/diffbot.ros2_control.xacro (robot description, xacro)
@@ -1,5 +1,5 @@
 <?xml version="1.0"?>
 <robot xmlns:xacro="http://www.ros.org/wiki/xacro">
-  <xacro:macro name="vcan_diffbot_ros2_control" params="name can_interface left_node_id right_node_id encoder_counts_per_revolution command_watchdog_ms feedback_timeout_ms">
+  <xacro:macro name="vcan_diffbot_ros2_control" params="name can_interface left_node_id right_node_id encoder_counts_per_revolution command_watchdog_ms ack_timeout_ms feedback_timeout_ms">
     <ros2_control name="${name}" type="system">
       <hardware>
@@ -10,4 +10,5 @@
         <param name="encoder_counts_per_revolution">${encoder_counts_per_revolution}</param>
         <param name="command_watchdog_ms">${command_watchdog_ms}</param>
+        <param name="ack_timeout_ms">${ack_timeout_ms}</param>
         <param name="feedback_timeout_ms">${feedback_timeout_ms}</param>
       </hardware>

File: src/vcan_diffbot_demo/urdf/diffbot.urdf.xacro (robot description, xacro)
@@ -6,4 +6,5 @@
   <xacro:arg name="encoder_counts_per_revolution" default="4096"/>
   <xacro:arg name="command_watchdog_ms" default="200"/>
+  <xacro:arg name="ack_timeout_ms" default="200"/>
   <xacro:arg name="feedback_timeout_ms" default="500"/>
   <xacro:property name="wheel_radius" value="0.10"/>
@@ -86,4 +87,5 @@
     encoder_counts_per_revolution="$(arg encoder_counts_per_revolution)"
     command_watchdog_ms="$(arg command_watchdog_ms)"
+    ack_timeout_ms="$(arg ack_timeout_ms)"
     feedback_timeout_ms="$(arg feedback_timeout_ms)"/>
 </robot>

Commit message: feat(canfd): add an opt-in versioned CAN-FD transport profile
The wire contract was classic 11-bit CAN at DLC 8 only. Add a CAN-FD profile
that is explicitly selected with transport:=canfd and keeps classic_can as the
default, so no existing deployment moves profiles by accident.

Every FD frame carries a version tag (byte 1) and a frame-type tag (byte 13),
and widens the request identity to a 32-bit command id plus a node id so a late
ACK stays attributable past an 8-bit sequence wrap. Decoders reject a wrong
version, a wrong frame type, an illegal data-phase length, and dirty reserved
bytes. Because the classic profile has no version field the two profiles cannot
be confused in either direction.

The sender and receiver are both opened for FD, and a socket opened for the
wrong profile fails configuration instead of silently downgrading. Payloads are
the same application fields as classic, so no physical throughput, latency or
electrical behaviour is claimed; the HIL recording procedure is documented
separately in both READMEs.

File: src/vcan_diffbot_demo/urdf/diffbot.ros2_control.xacro (robot description, xacro)
@@ -1,5 +1,5 @@
 <?xml version="1.0"?>
 <robot xmlns:xacro="http://www.ros.org/wiki/xacro">
-  <xacro:macro name="vcan_diffbot_ros2_control" params="name can_interface left_node_id right_node_id encoder_counts_per_revolution command_watchdog_ms ack_timeout_ms feedback_timeout_ms">
+  <xacro:macro name="vcan_diffbot_ros2_control" params="name can_interface left_node_id right_node_id encoder_counts_per_revolution command_watchdog_ms ack_timeout_ms feedback_timeout_ms transport:=classic_can brs:=auto">
     <ros2_control name="${name}" type="system">
       <hardware>
@@ -12,4 +12,6 @@
         <param name="ack_timeout_ms">${ack_timeout_ms}</param>
         <param name="feedback_timeout_ms">${feedback_timeout_ms}</param>
+        <param name="transport">${transport}</param>
+        <param name="brs">${brs}</param>
       </hardware>
       <joint name="left_wheel_joint">
